File: pcb/rev.KA2/zx-multisound.kicad_pcb (KiCad board)
At the start: 2 copper layers, 170 x 64 mm, 198 parts, among them J1 PJ307, J2 Conn_01x04, J3 Conn_01x04, J4 Conn_02x30_Row_Letter_First, J5 Conn_02x05_Odd_Even, SW1 SW_DIP_x05, U1 LM358D, U10 YM2203, U11 27C512, U12 YM3014B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

Commit message: Added label about SW[4]
Other:
- board text added: "SW1.1 - Enable TSFM + MIDI SW1.2 - Enable SAA1099 SW1.3 - Enable GS SW1.4 - Enable SounDrive SW1.5 - Enable Beeper"
- board text removed: "SW1.1 - Enable TSFM + MIDI SW1.2 - Enable SAA1099 SW1.3 - Enable GS SW1.4 - Enable SounDrive SW1.5 - Reserved"
Changed lines of the file:
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@@
 		)
 	)
-	(gr_text "SW1.1 - Enable TSFM + MIDI\nSW1.2 - Enable SAA1099\nSW1.3 - Enable GS\nSW1.4 - Enable SounDrive\nSW1.5 - Reserved"
+	(gr_text "SW1.1 - Enable TSFM + MIDI\nSW1.2 - Enable SAA1099\nSW1.3 - Enable GS\nSW1.4 - Enable SounDrive\nSW1.5 - Enable Beeper"
 		(at 178.15 79.35 0)
 		(layer "B.SilkS")
